File: gloves/kiya/PCB/kaya-insolev1.brd (EAGLE design)
At the start: 160 x 100 mm, 16 parts, among them U1 LSM9DS1, U2 MCP73832T-2ACI/OT

Commit message: PCB v1
Parts:
- added LED1: (no value), led:CHIPLED_0603
- added R4: (no value), rcl:R0603
- moved BAT 53.6 mm to (30.5, 33.0), turned to 0 degrees
- moved U2 53.4 mm to (52.1, 44.5)
- moved C6 52.3 mm to (43.2, 34.3), turned to 0 degrees
- moved C1 50.1 mm to (52.1, 40.6), turned to 180 degrees
- moved C2 49.5 mm to (55.9, 49.5), turned to 90 degrees
- moved R1 47.1 mm to (52.1, 49.5)
- moved R3 46.7 mm to (43.2, 48.3), turned to 270 degrees
- moved C3 45.5 mm to (43.2, 39.4), turned to 0 degrees
- moved C7 45.5 mm to (43.2, 44.5), turned to 0 degrees
- moved R2 40.7 mm to (43.2, 54.6)
- moved SV2 34.9 mm to (30.5, 58.4), turned to 180 degrees
- moved C5 30.5 mm to (16.5, 50.8)
- moved U$1 28.4 mm to (30.5, 43.2)
- moved C4 28.2 mm to (12.7, 50.8), turned to 270 degrees
- moved J1 19.0 mm to (2.54, 43.2), flipped to the top, turned to 0 degrees
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Connections:
- net D+ renamed TXD
- net D- renamed RXD
- net N$2 renamed GND
- new net N$11: C2.2, J1.GND, R1.1, U2.2
- new net N$12: BAT.3, C1.1, C2.1, U2.3
- net N$1: now also C1.2, J1.VBUS, LED1.A, U2.4; no longer C1.1, C2.1, C2.2, J1.GND, R1.1, U2.2
- net N$8: now also LED1.C, R4.2; no longer C1.2, J1.VBUS, U2.4
- net N$9: now also R4.1, U2.1; no longer BAT.3, U2.3
Routing:
- net GND: track 89.1 -> 0.00 mm, vias 1 -> 0
- net N$14: track 52.4 -> 0.00 mm
- net N$1: track 47.4 -> 0.00 mm
- net VIN: track 46.8 -> 0.00 mm
- net N$13: track 42.6 -> 0.00 mm
- net N$7: track 33.0 -> 0.00 mm
- net TXD: track 28.0 -> 0.00 mm, vias 1 -> 0
- net N$3: track 19.2 -> 0.00 mm
- net N$4: track 18.5 -> 0.00 mm
- net VDD: track 18.0 -> 0.00 mm, vias 1 -> 0
- net N$9: track 9.78 -> 0.00 mm
- net N$6: track 8.20 -> 0.00 mm, vias 2 -> 0
- net N$8: track 7.38 -> 0.00 mm, vias 2 -> 0
- net N$16: track 5.98 -> 0.00 mm
- net N$5: track 4.48 -> 0.00 mm
