File: gloves/kiya/PCB/kaya-insolev1.sch (EAGLE design)
At the start: 16 parts, among them U1 LSM9DS1, U2 MCP73832T-2ACI/OT

Commit message: PCB v1
Parts:
- added LED1: (no value), led:LEDCHIPLED_0603
- added R4: (no value), rcl:R-EU_R0603
Connections:
- net D+ renamed TXD
- net D- renamed RXD
- net N$2 renamed GND
- new net N$11: C2.22, J1.GND, R1.11, U2.VSS
- new net N$12: BAT.3, C1.11, C2.11, U2.VBAT
- net N$1: now also C1.22, J1.VBUS, LED1.A, U2.VDD; no longer C1.11, C2.11, C2.22, J1.GND, R1.11, U2.VSS
- net N$8: now also LED1.C, R4.2; no longer C1.22, J1.VBUS, U2.VDD
- net N$9: now also R4.1, U2.STAT; no longer BAT.3, U2.VBAT
Other:
- moved on the sheet: BAT, C1, C2, C3, C4, C5, C6, C7, J1, R1, R2, R3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

Commit message: routing complete
Connections:
- net N$1 renamed VBUS
- removed net N$11: C2.22, J1.GND, R1.11, U2.VSS
- net GND: now also C2.22, J1.GND, R1.11, U2.VSS
- net N$13: now also SV2.1; no longer SV2.2
- net N$14: now also SV2.2; no longer SV2.1
Changed lines of the file:
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@@
 <?xml version="1.0" encoding="utf-8"?>
 <!DOCTYPE eagle SYSTEM "eagle.dtd">
-<eagle version="8.5.0">
+<eagle version="8.6.0">
 <drawing>
 <settings>
@@
 <instances>
 <instance part="U1" gate="G$1" x="-27.94" y="91.44"/>
-<instance part="U2" gate="G$1" x="-38.1" y="30.48"/>
+<instance part="U2" gate="G$1" x="-38.1" y="30.48" smashed="yes">
+<attribute name="NAME" x="-53.3713" y="15.2087" size="1.781659375" layer="95"/>
+<attribute name="VALUE" x="-53.3586" y="12.6784" size="1.780159375" layer="96"/>
+</instance>
 <instance part="R1" gate="A" x="-33.02" y="43.18" rot="R180"/>
 <instance part="C1" gate="A" x="-50.8" y="5.08"/>
@@
 <net name="N$13" class="0">
 <segment>
-<pinref part="SV2" gate="G$1" pin="2"/>
-<wire x1="-93.98" y1="-43.18" x2="-81.28" y2="-43.18" width="0.1524" layer="91"/>
-<wire x1="-81.28" y1="-43.18" x2="-81.28" y2="-38.1" width="0.1524" layer="91"/>
 <pinref part="R2" gate="A" pin="22"/>
-<wire x1="-81.28" y1="-38.1" x2="-68.58" y2="-38.1" width="0.1524" layer="91"/>
+<wire x1="-83.82" y1="-38.1" x2="-68.58" y2="-38.1" width="0.1524" layer="91"/>
 <wire x1="-68.58" y1="-38.1" x2="-68.58" y2="-25.4" width="0.1524" layer="91"/>
 <junction x="-68.58" y="-38.1"/>
@@
 <pinref part="U$1" gate="G$1" pin="A3"/>
 <wire x1="106.68" y1="95.78" x2="52.46" y2="95.78" width="0.1524" layer="91"/>
+<wire x1="-83.82" y1="-38.1" x2="-83.82" y2="-45.72" width="0.1524" layer="91"/>
+<pinref part="SV2" gate="G$1" pin="1"/>
+<wire x1="-83.82" y1="-45.72" x2="-93.98" y2="-45.72" width="0.1524" layer="91"/>
 </segment>
 </net>
 <net name="N$14" class="0">
 <segment>
-<pinref part="SV2" gate="G$1" pin="1"/>
 <pinref part="R3" gate="A" pin="22"/>
-<wire x1="-93.98" y1="-45.72" x2="-68.58" y2="-45.72" width="0.1524" layer="91"/>
 <wire x1="-68.58" y1="-45.72" x2="-68.58" y2="-48.26" width="0.1524" layer="91"/>
 <wire x1="-68.58" y1="-48.26" x2="-68.58" y2="-60.96" width="0.1524" layer="91"/>
@@
 <wire x1="86.36" y1="-60.96" x2="86.36" y2="91.44" width="0.1524" layer="91"/>
 <wire x1="86.36" y1="91.44" x2="52.46" y2="91.44" width="0.1524" layer="91"/>
-</segment>
-</net>
-<net name="N$1" class="0">
+<wire x1="-68.58" y1="-45.72" x2="-78.74" y2="-45.72" width="0.1524" layer="91"/>
+<wire x1="-78.74" y1="-45.72" x2="-78.74" y2="-43.18" width="0.1524" layer="91"/>
+<pinref part="SV2" gate="G$1" pin="2"/>
+<wire x1="-78.74" y1="-43.18" x2="-93.98" y2="-43.18" width="0.1524" layer="91"/>
+</segment>
+</net>
+<net name="VBUS" class="0">
 <segment>
 <pinref part="J1" gate="G$1" pin="VBUS"/>
@@
 </segment>
 </net>
-<net name="N$11" class="0">
-<segment>
-<pinref part="J1" gate="G$1" pin="GND"/>
-<wire x1="-93.98" y1="25.4" x2="-83.82" y2="25.4" width="0.1524" layer="91"/>
-<wire x1="-83.82" y1="25.4" x2="-83.82" y2="30.48" width="0.1524" layer="91"/>
-<pinref part="U2" gate="G$1" pin="VSS"/>
-<wire x1="-83.82" y1="30.48" x2="-60.96" y2="30.48" width="0.1524" layer="91"/>
-<pinref part="C2" gate="A" pin="22"/>
-<wire x1="-60.96" y1="30.48" x2="-53.34" y2="30.48" width="0.1524" layer="91"/>
-<junction x="-60.96" y="30.48"/>
-<pinref part="R1" gate="A" pin="11"/>
-<wire x1="-45.72" y1="43.18" x2="-53.34" y2="43.18" width="0.1524" layer="91"/>
-<wire x1="-53.34" y1="43.18" x2="-53.34" y2="30.48" width="0.1524" layer="91"/>
-<junction x="-53.34" y="30.48"/>
-</segment>
-</net>
 <net name="N$12" class="0">
 <segment>
@@
 <wire x1="-78.74" y1="73.66" x2="-58.42" y2="73.66" width="0.1524" layer="91"/>
 <pinref part="C7" gate="G$1" pin="2"/>
-<wire x1="-104.14" y1="73.66" x2="-58.42" y2="73.66" width="0.1524" layer="91"/>
+<wire x1="-104.14" y1="73.66" x2="-99.06" y2="73.66" width="0.1524" layer="91"/>
 <pinref part="C6" gate="G$1" pin="2"/>
+<wire x1="-99.06" y1="73.66" x2="-58.42" y2="73.66" width="0.1524" layer="91"/>
 <wire x1="-91.44" y1="73.66" x2="-58.42" y2="73.66" width="0.1524" layer="91"/>
 <pinref part="U$1" gate="G$1" pin="GND"/>
@@
 <wire x1="-55.88" y1="-48.26" x2="18.86" y2="-48.26" width="0.1524" layer="91"/>
 <wire x1="18.86" y1="-48.26" x2="18.86" y2="82.76" width="0.1524" layer="91"/>
+<wire x1="-99.06" y1="73.66" x2="-99.06" y2="53.34" width="0.1524" layer="91"/>
+<wire x1="-99.06" y1="53.34" x2="-116.84" y2="53.34" width="0.1524" layer="91"/>
+<junction x="-99.06" y="73.66"/>
+<wire x1="-116.84" y1="53.34" x2="-116.84" y2="17.78" width="0.1524" layer="91"/>
+<wire x1="-116.84" y1="17.78" x2="-86.36" y2="17.78" width="0.1524" layer="91"/>
+<pinref part="J1" gate="G$1" pin="GND"/>
+<wire x1="-93.98" y1="25.4" x2="-86.36" y2="25.4" width="0.1524" layer="91"/>
+<wire x1="-86.36" y1="25.4" x2="-83.82" y2="25.4" width="0.1524" layer="91"/>
+<wire x1="-83.82" y1="25.4" x2="-83.82" y2="30.48" width="0.1524" layer="91"/>
+<pinref part="U2" gate="G$1" pin="VSS"/>
+<wire x1="-83.82" y1="30.48" x2="-60.96" y2="30.48" width="0.1524" layer="91"/>
+<pinref part="C2" gate="A" pin="22"/>
+<wire x1="-60.96" y1="30.48" x2="-53.34" y2="30.48" width="0.1524" layer="91"/>
+<junction x="-60.96" y="30.48"/>
+<pinref part="R1" gate="A" pin="11"/>
+<wire x1="-45.72" y1="43.18" x2="-53.34" y2="43.18" width="0.1524" layer="91"/>
+<wire x1="-53.34" y1="43.18" x2="-53.34" y2="30.48" width="0.1524" layer="91"/>
+<junction x="-53.34" y="30.48"/>
+<wire x1="-86.36" y1="17.78" x2="-86.36" y2="25.4" width="0.1524" layer="91"/>
+<junction x="-86.36" y="25.4"/>
 </segment>
 </net>
@@
 </sheet>
 </sheets>
+<errors>
+</errors>
 </schematic>
 </drawing>
