File: gloves/kiya/PCB/nicks junk/kaya-insolev1.brd (EAGLE design)
At the start: 100 x 80 mm, 16 parts, among them U1 LSM9DS1, U2 MCP73832T-2ACI/OT

Commit message: nii
Routing:
- net N$14: track 58.1 -> 0.00 mm
- net N$2: track 56.5 -> 2.71 mm
- net VIN: track 51.9 -> 0.07 mm
- net N$13: track 48.4 -> 0.00 mm, vias 2 -> 0
- net VDD: track 42.6 -> 0.00 mm
- net D+: track 37.3 -> 0.00 mm, vias 2 -> 0
- net N$7: track 23.3 -> 0.00 mm, vias 4 -> 0
- net N$8: track 13.0 -> 0.00 mm
- net N$1: track 12.9 -> 0.00 mm
- net N$6: track 11.7 -> 0.00 mm
- net N$4: track 11.2 -> 0.00 mm
- net N$5: track 9.96 -> 0.00 mm
- net N$9: track 9.92 -> 0.00 mm
- net N$3: track 8.55 -> 0.00 mm
- net N$11: track 1.79 -> 0.00 mm
