File: PCB/Kaya.sch (EAGLE design)
At the start: 23 parts, among them U1 MCP73832T-2ACI/OT, U2 LSM9DS1

Commit message: Finished PCB
Parts:
- added PAD1, PAD2: WIREPADSMD1,27-254, wirepad:WIREPADSMD1,27-254
Connections:
- new net N$10: PAD1.P, U$1.IN_R
- new net N$11: PAD2.P, U$1.IN_L
Changed lines of the file:
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@@
 <part name="U$4" library="tex-tronics" deviceset="CONDUCTIVE-BUTTON" device=""/>
 <part name="U$5" library="tex-tronics" deviceset="CONDUCTIVE-BUTTON" device=""/>
+<part name="PAD1" library="wirepad" library_urn="urn:adsk.eagle:library:412" deviceset="WIREPAD" device="SMD1,27-254" package3d_urn="urn:adsk.eagle:package:30839/1"/>
+<part name="PAD2" library="wirepad" library_urn="urn:adsk.eagle:library:412" deviceset="WIREPAD" device="SMD1,27-254" package3d_urn="urn:adsk.eagle:package:30839/1"/>
 </parts>
 <sheets>
@@
 <instance part="GND4" gate="1" x="172.72" y="30.48"/>
 <instance part="GND5" gate="1" x="187.96" y="30.48"/>
+<instance part="PAD1" gate="G$1" x="12.7" y="91.44"/>
+<instance part="PAD2" gate="G$1" x="12.7" y="81.28"/>
 </instances>
 <busses>
@@
 </segment>
 </net>
+<net name="N$10" class="0">
+<segment>
+<pinref part="PAD1" gate="G$1" pin="P"/>
+<pinref part="U$1" gate="INDUCTIVE-5V" pin="IN_R"/>
+<wire x1="15.24" y1="91.44" x2="33.02" y2="91.44" width="0.1524" layer="91"/>
+</segment>
+</net>
+<net name="N$11" class="0">
+<segment>
+<pinref part="PAD2" gate="G$1" pin="P"/>
+<pinref part="U$1" gate="INDUCTIVE-5V" pin="IN_L"/>
+<wire x1="15.24" y1="81.28" x2="33.02" y2="81.28" width="0.1524" layer="91"/>
+</segment>
+</net>
