File: PCB/version1/PCB/kaya-insolev1.brd (EAGLE design)
At the start: 47.6 x 25.7 mm, 18 parts, among them U1 LSM9DS1, U2 MCP73832T-2ACI/OT

Commit message: LPKF READY FILES
Readjusted design check for the new machine
Connections:
- net N$12 renamed VBAT
- removed net N$7: C3.1, C6.1, C7.1, U$1.VDD, U1.1, U1.22, U1.23, U1.3
- net VDD: now also C3.1, C6.1, C7.1, U$1.VDD, U1.1, U1.22, U1.23, U1.3
Routing:
- net VDD: track 17.9 -> 48.0 mm, vias 0 -> 2
- net N$7: track 29.1 -> 0.00 mm
- net VIN: track 1.86 -> 28.8 mm, vias 1 -> 2
- net GND: track 97.7 -> 84.4 mm, vias 1 -> 3
- net N$14: track 54.3 -> 62.1 mm, vias 0 -> 2
Other:
- outline, holes or cut-outs redrawn
