File: PCB/version1/PCB/kaya-insolev1.sch (EAGLE design)
At the start: 18 parts, among them U1 LSM9DS1, U2 MCP73832T-2ACI/OT

Commit message: LPKF READY FILES
Readjusted design check for the new machine
Connections:
- net N$12 renamed VBAT
- removed net N$7: C3.1, C6.1, C7.1, U$1.VDD, U1.VDD, U1.VDDIO
- net VDD: now also C3.1, C6.1, C7.1, U$1.VDD, U1.VDD, U1.VDDIO
Changed lines of the file:
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@@
 <?xml version="1.0" encoding="utf-8"?>
 <!DOCTYPE eagle SYSTEM "eagle.dtd">
-<eagle version="8.5.0">
+<eagle version="9.1.2">
 <drawing>
 <settings>
@@
 <wire x1="-93.98" y1="-40.64" x2="-91.44" y2="-40.64" width="0.1524" layer="91"/>
 </segment>
-</net>
-<net name="N$5" class="0">
-<segment>
-<pinref part="U1" gate="G$1" pin="C1"/>
-<pinref part="C4" gate="G$1" pin="1"/>
-<wire x1="-43.18" y1="96.52" x2="-58.42" y2="96.52" width="0.1524" layer="91"/>
-<wire x1="-58.42" y1="96.52" x2="-58.42" y2="81.28" width="0.1524" layer="91"/>
-</segment>
-</net>
-<net name="N$6" class="0">
-<segment>
-<pinref part="U1" gate="G$1" pin="CAP"/>
-<pinref part="C5" gate="G$1" pin="1"/>
-<wire x1="-43.18" y1="99.06" x2="-68.58" y2="99.06" width="0.1524" layer="91"/>
-<wire x1="-68.58" y1="99.06" x2="-68.58" y2="81.28" width="0.1524" layer="91"/>
-</segment>
-</net>
-<net name="N$7" class="0">
 <segment>
 <pinref part="U1" gate="G$1" pin="VDDIO"/>
@@
 </segment>
 </net>
+<net name="N$5" class="0">
+<segment>
+<pinref part="U1" gate="G$1" pin="C1"/>
+<pinref part="C4" gate="G$1" pin="1"/>
+<wire x1="-43.18" y1="96.52" x2="-58.42" y2="96.52" width="0.1524" layer="91"/>
+<wire x1="-58.42" y1="96.52" x2="-58.42" y2="81.28" width="0.1524" layer="91"/>
+</segment>
+</net>
+<net name="N$6" class="0">
+<segment>
+<pinref part="U1" gate="G$1" pin="CAP"/>
+<pinref part="C5" gate="G$1" pin="1"/>
+<wire x1="-43.18" y1="99.06" x2="-68.58" y2="99.06" width="0.1524" layer="91"/>
+<wire x1="-68.58" y1="99.06" x2="-68.58" y2="81.28" width="0.1524" layer="91"/>
+</segment>
+</net>
 <net name="N$13" class="0">
 <segment>
@@
 </segment>
 </net>
-<net name="N$12" class="0">
+<net name="VBAT" class="0">
 <segment>
 <pinref part="C2" gate="A" pin="11"/>
