File: PCB/version1.2/PCB/kaya-insolev1.brd (EAGLE design)
At the start: 31.9 x 25.5 mm, 18 parts, among them U1 LSM9DS1, U2 MCP

Commit message: LPKF READY FILES
Readjusted design check for the new machine
Routing:
- net GND: vias 9 -> 8
Other:
- outline, holes or cut-outs redrawn
Changed lines of the file:
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@@
 <?xml version="1.0" encoding="utf-8"?>
 <!DOCTYPE eagle SYSTEM "eagle.dtd">
-<eagle version="9.1.2">
+<eagle version="9.1.0">
 <drawing>
 <settings>
@@
 <layer number="43" name="vRestrict" color="2" fill="10" visible="no" active="yes"/>
 <layer number="44" name="Drills" color="7" fill="1" visible="no" active="yes"/>
-<layer number="45" name="Holes" color="7" fill="1" visible="no" active="yes"/>
+<layer number="45" name="Holes" color="7" fill="1" visible="yes" active="yes"/>
 <layer number="46" name="Milling" color="3" fill="1" visible="no" active="yes"/>
 <layer number="47" name="Measures" color="7" fill="1" visible="no" active="yes"/>
@@
 <rectangle x1="115.57" y1="49.53" x2="128.397" y2="63.881" layer="42"/>
 <rectangle x1="115.57" y1="49.53" x2="128.397" y2="63.881" layer="45"/>
-<dimension x1="104.267" y1="43.434" x2="136.652" y2="43.434" x3="120.4595" y3="35.941" textsize="0.254" layer="45"/>
-<dimension x1="110.236" y1="64.516" x2="110.617" y2="38.354" x3="100.203" y3="51.435" textsize="0.254" layer="45" dtype="vertical"/>
-<dimension x1="103.886" y1="65.278" x2="136.652" y2="52.705" x3="120.269" y3="67.056" textsize="1.778" layer="1" dtype="horizontal" unit="inch"/>
-<dimension x1="104.013" y1="64.516" x2="110.744" y2="38.481" x3="97.663" y3="51.4985" textsize="1.778" layer="1" dtype="vertical" unit="inch"/>
+<wire x1="115.57" y1="63.627" x2="115.57" y2="49.657" width="0.1524" layer="20"/>
+<wire x1="115.57" y1="49.657" x2="115.697" y2="49.53" width="0.1524" layer="20"/>
+<wire x1="115.697" y1="49.53" x2="128.27" y2="49.53" width="0.1524" layer="20"/>
+<wire x1="128.27" y1="49.53" x2="128.27" y2="63.627" width="0.1524" layer="20"/>
+<wire x1="128.27" y1="63.627" x2="128.27" y2="63.881" width="0.1524" layer="20"/>
+<wire x1="128.27" y1="63.881" x2="115.697" y2="63.881" width="0.1524" layer="20"/>
+<wire x1="115.697" y1="63.881" x2="115.57" y2="63.754" width="0.1524" layer="20"/>
+<wire x1="115.57" y1="63.754" x2="115.57" y2="63.627" width="0.1524" layer="20"/>
 </plain>
 <attributes>
@@
 <param name="mtCopper" value="0.035mm 0.035mm 0.035mm 0.035mm 0.035mm 0.035mm 0.035mm 0.035mm 0.035mm 0.035mm 0.035mm 0.035mm 0.035mm 0.035mm 0.035mm 0.035mm"/>
 <param name="mtIsolate" value="0.2mm 0.15mm 0.2mm 0.15mm 0.2mm 0.15mm 0.2mm 0.15mm 0.2mm 0.15mm 0.2mm 0.15mm 0.2mm 0.15mm 0.2mm"/>
-<param name="mdWireWire" value="6mil"/>
-<param name="mdWirePad" value="6mil"/>
-<param name="mdWireVia" value="6mil"/>
-<param name="mdPadPad" value="6mil"/>
-<param name="mdPadVia" value="6mil"/>
-<param name="mdViaVia" value="6mil"/>
+<param name="mdWireWire" value="5mil"/>
+<param name="mdWirePad" value="5mil"/>
+<param name="mdWireVia" value="5mil"/>
+<param name="mdPadPad" value="5mil"/>
+<param name="mdPadVia" value="5mil"/>
+<param name="mdViaVia" value="5mil"/>
 <param name="mdSmdPad" value="5mil"/>
 <param name="mdSmdVia" value="5mil"/>
@@
 <param name="mdViaViaSameLayer" value="6mil"/>
 <param name="mnLayersViaInSmd" value="2"/>
-<param name="mdCopperDimension" value="10mil"/>
-<param name="mdDrill" value="6mil"/>
+<param name="mdCopperDimension" value="2mil"/>
+<param name="mdDrill" value="8mil"/>
 <param name="mdSmdStop" value="0mil"/>
 <param name="msWidth" value="5mil"/>
-<param name="msDrill" value="0.15mm"/>
+<param name="msDrill" value="0.2mm"/>
 <param name="msMicroVia" value="100mm"/>
 <param name="msBlindViaRatio" value="0.5"/>
@@
 <vertex x="103.632" y="65.024"/>
 </polygon>
-<via x="112.522" y="54.737" extent="1-2" drill="0.127" diameter="0.00761875"/>
+<wire x1="114.717203125" y1="45.72" x2="127" y2="44.45" width="0" layer="19" extent="1-1"/>
+<wire x1="114.264" y1="43.18" x2="114.717203125" y2="45.72" width="0" layer="19" extent="1-1"/>
+<wire x1="110.49" y1="50.8" x2="114.17" y2="49.84" width="0" layer="19" extent="1-1"/>
+<wire x1="107.715" y1="57.195" x2="107.95" y2="53.76" width="0" layer="19" extent="1-1"/>
+<wire x1="106.68" y1="63.08" x2="107.745" y2="59.065" width="0" layer="19" extent="1-1"/>
 </signal>
 <signal name="VIN">

Commit message: wirechange
Connections:
- net GND: now also C1.1
- net N$12: no longer C1.1
Routing:
- net N$12: track 11.0 -> 7.77 mm
Changed lines of the file:
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@@
 <contactref element="C2" pad="1"/>
 <contactref element="U2" pad="3"/>
-<contactref element="C1" pad="1"/>
 <contactref element="BAT" pad="3"/>
 <wire x1="111.76" y1="41.0845" x2="112.2045" y2="40.64" width="0.254" layer="1"/>
-<wire x1="112.2045" y1="40.64" x2="114.7445" y2="40.64" width="0.254" layer="1"/>
-<wire x1="114.7445" y1="40.64" x2="114.264" y2="41.1205" width="0.254" layer="1"/>
 <wire x1="114.264" y1="41.1205" x2="114.264" y2="42.23" width="0.254" layer="1"/>
 <wire x1="114.264" y1="42.23" x2="114.6346" y2="42.6006" width="0.254" layer="1"/>
@@
 <wire x1="115.92973125" y1="43.5506" x2="117.59173125" y2="43.5506" width="0.254" layer="1"/>
 <wire x1="114.97973125" y1="42.6006" x2="115.92973125" y2="43.5506" width="0.254" layer="1"/>
+<wire x1="114.264" y1="41.1205" x2="112.2045" y2="40.64" width="0" layer="19" extent="1-1"/>
 </signal>
 <signal name="N$16">
@@
 <vertex x="103.632" y="65.024"/>
 </polygon>
+<contactref element="C1" pad="1"/>
 <wire x1="114.717203125" y1="45.72" x2="127" y2="44.45" width="0" layer="19" extent="1-1"/>
 <wire x1="114.264" y1="43.18" x2="114.717203125" y2="45.72" width="0" layer="19" extent="1-1"/>
+<wire x1="114.7445" y1="40.64" x2="113.03" y2="41.91" width="0" layer="19" extent="1-1"/>
 <wire x1="110.49" y1="50.8" x2="114.17" y2="49.84" width="0" layer="19" extent="1-1"/>
 <wire x1="107.715" y1="57.195" x2="107.95" y2="53.76" width="0" layer="19" extent="1-1"/>
